File: hardware/eeg.kicad_pcb (KiCad board)
At the start: 4 copper layers, 67.3 x 41.7 mm, 147 parts, among them IC1 TPS62162QDSGRQ1, IC2 LT3042IMSE#PBF, IC3 STM32H730VBT6, IC4 OPA333AIDCKRG4, J1 Battery LiPO, J2 Conn_01x05, J4 Serial, SW2 SW_Push_Dual, SW3 SW_Push_Dual, U1 INA333xxDRG, U10 OPA333xxDCK, U11 MCP602, U12 MCP602, U17 OPA333xxDCK, U18 OPA333xxDCK, U19 OPA333xxDCK, U2 OPA333xxDCK, U3 MCP602, U4 MCP602, U5 INA333xxDRG, U6 OPA333xxDCK, U7 MCP602, U8 MCP602, U9 INA333xxDRG, Y1 Crystal_GND24_Small

Commit message: Hardware att
Other:
- board text removed: "Stephan C. Barros stephanbrrs8@gmail.com"
Changed lines of the file:
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@@
-		)
-	)
-	(gr_text "Stephan C. Barros\nstephanbrrs8@gmail.com\n\n "
-		(at 163.81 95.23 0)
-		(layer "B.SilkS")
-		(effects
-			(font
-				(size 0.8 0.8)
-				(thickness 0.2)
-				(bold yes)
-				(italic yes)
-			)
-			(justify left bottom mirror)
 		)
 	)
