File: hardware/eeg.kicad_sch (KiCad schematic)
At the start: 152 parts, among them IC1 TPS62162QDSGRQ1, IC10 INA333AIDRGT, IC11 OPA333AIDCKRG4, IC12 MCP602-E_SN, IC13 MCP602-E_SN, IC14 INA333AIDRGT, IC15 OPA333AIDCKRG4, IC16 MCP602-E_SN, IC17 MCP602-E_SN, IC18 INA333AIDRGT, IC19 OPA333AIDCKRG4, IC2 LT3042IMSE#PBF, IC20 MCP602-E_SN, IC21 MCP602-E_SN, IC22 OPA333AIDCKRG4, IC3 STM32H730VBT6, IC4 ESP32-C6-MINI-1-H4, IC5 W25Q512JVFIQ, IC6 INA333AIDRGT, IC7 OPA333AIDCKRG4, IC8 MCP602-E_SN, IC9 MCP602-E_SN, J1 Battery LiPO, J2 USB4105-GF-A, J3 ST-Link, J4 Serial, J5 Serial, SW1 SW_Push_Dual, SW2 SW_Push_Dual, SW3 SW_Push_Dual, U1 USBLC6-2SC6, Y1 Crystal_GND24_Small, Y2 Crystal_GND24_Small

Commit message: hardware final update
Parts:
- removed C1: 10uF, Capacitor_SMD:C_0402_1005Metric, symbol Device:C
- removed C2, C24: 22uF, Capacitor_SMD:C_0402_1005Metric, symbol Device:C
- removed C21, C22: 20pF, Capacitor_SMD:C_0402_1005Metric, symbol Device:C
- removed C23: 1uF, Capacitor_SMD:C_0402_1005Metric, symbol Device:C
- removed C25, C26, C27, C35, C36, C44, C45, C53, C54: 0.1uF, Capacitor_SMD:C_0402_1005Metric, symbol Device:C
- removed C28, C37, C46, C55: 330nF, Capacitor_SMD:C_0402_1005Metric, symbol Device:C
- removed C29, C30, C38, C39, C47, C48, C56, C57: 36nF, Capacitor_SMD:C_0402_1005Metric, symbol Device:C
- removed C3, C5: 4.7uF, Capacitor_SMD:C_0402_1005Metric, symbol Device:C
- removed C31, C40, C49, C58: 8.2nF, Capacitor_SMD:C_0402_1005Metric, symbol Device:C
- removed C32, C33, C34, C41, C42, C43, C50, C51, C52, C59, C60, C61: 300nF, Capacitor_SMD:C_0402_1005Metric, symbol Device:C
- removed C4: 0.47uF, Capacitor_SMD:C_0402_1005Metric, symbol Device:C
- removed D1: LED, LED_SMD:LED_0402_1005Metric, symbol Device:LED
- removed FB1: FerriteBead_Small, ferritebead:BEADC1005X55N, symbol Device:FerriteBead_Small
- removed IC1: TPS62162QDSGRQ1, tps62162:SON50P200X200X80-9N, symbol TPS62162QDSGRQ1:TPS62162QDSGRQ1
- removed IC10, IC14, IC18, IC6: INA333AIDRGT, ina333:SON50P300X300X80-9N-D, symbol INA333AIDRGT:INA333AIDRGT
- removed IC11, IC15, IC19, IC22, IC7: OPA333AIDCKRG4, opa333:SOT65P210X110-5N, symbol OPA333AIDCKRG4:OPA333AIDCKRG4
- removed IC12, IC13, IC16, IC17, IC20, IC21, IC8, IC9: MCP602-E_SN, mcp602:SOIC127P600X175-8N, symbol MCP602-E_SN:MCP602-E_SN
- removed IC2: LT3042IMSE#PBF, lt3042:SOP50P490X110-11N, symbol LT3042IMSE#PBF:LT3042IMSE#PBF
- removed IC4: ESP32-C6-MINI-1-H4, esp32c6:ESP32C6MINI1H4, symbol ESP32-C6-MINI-1-H4:ESP32-C6-MINI-1-H4
- removed IC5: W25Q512JVFIQ, w25q512jvfiq:SOIC127P1032X264-16N, symbol W25Q512JVFIQ:W25Q512JVFIQ
- removed J1: Battery LiPO, Connector_PinHeader_2.54mm:PinHeader_1x02_P2.54mm_Vertical, symbol Connector_Generic:Conn_01x02
- removed J2: USB4105-GF-A, usb_otg:GCT_USB4105-GF-A, symbol USB4105-GF-A:USB4105-GF-A
- removed J4, J5: Serial, Connector_PinHeader_2.54mm:PinHeader_1x04_P2.54mm_Vertical, symbol Connector_Generic:Conn_01x04
- removed JP1: Jumper_2_Bridged, Jumper:SolderJumper-2_P1.3mm_Open_Pad1.0x1.5mm, symbol Jumper:Jumper_2_Bridged
- removed L1: 2.2uH, Inductor_SMD:L_0402_1005Metric, symbol Device:L
- removed R0: 100k, Resistor_SMD:R_0402_1005Metric, symbol Device:R
- removed R1: 33.2k, Resistor_SMD:R_0402_1005Metric, symbol Device:R
- removed R10, R20, R30: 910k, Resistor_SMD:R_0402_1005Metric, symbol Device:R
- removed R11, R21, R31: 1.5k, Resistor_SMD:R_0402_1005Metric, symbol Device:R
- removed R12, R22, R32, R42: 750k, Resistor_SMD:R_0402_1005Metric, symbol Device:R
- removed R13, R23, R33, R43: 97k, Resistor_SMD:R_0402_1005Metric, symbol Device:R
- removed R14, R24, R34, R44: 149K, Resistor_SMD:R_0402_1005Metric, symbol Device:R
- removed R15, R25, R35, R45: 276K, Resistor_SMD:R_0402_1005Metric, symbol Device:R
- removed R16, R26, R36, R46: 967k, Resistor_SMD:R_0402_1005Metric, symbol Device:R
- removed R17, R27, R37, R47: 484k, Resistor_SMD:R_0402_1005Metric, symbol Device:R
- removed R18, R28, R38, R48: 1.93M, Resistor_SMD:R_0402_1005Metric, symbol Device:R
- removed R19, R29, R9: 5.26k, Resistor_SMD:R_0402_1005Metric, symbol Device:R
- removed R4, R52: 1k, Resistor_SMD:R_0402_1005Metric, symbol Device:R
- removed R49: 5.2k, Resistor_SMD:R_0402_1005Metric, symbol Device:R
- removed R5, R50, R51, R6, R7, R8: 10k, Resistor_SMD:R_0402_1005Metric, symbol Device:R
- removed S1: PCM12SMTBR, sw_tactile:PCM12SMTBR, symbol PCM12SMTBR:PCM12SMTBR
- removed SW1: SW_Push_Dual, tactile_button:TL1030AF160BQJ, symbol Switch:SW_Push_Dual
- removed U1: USBLC6-2SC6, Package_TO_SOT_SMD:SOT-23-6, symbol Power_Protection:USBLC6-2SC6
- removed Y2: Crystal_GND24_Small, crystal30M:830107284409, symbol Device:Crystal_GND24_Small
- added D2, D3, D4: LED, LED_SMD:LED_0402_1005Metric, symbol Device:LED
- added J4: Serial, Connector_PinHeader_2.54mm:PinHeader_1x03_P2.54mm_Vertical, symbol Connector_Generic:Conn_01x03
- C30: renamed from C11; footprint Capacitor_SMD:C_0402_1005Metric -> Capacitor_SMD:C_0603_1608Metric
- C36: renamed from C17; footprint Capacitor_SMD:C_0402_1005Metric -> Capacitor_SMD:C_0603_1608Metric
- R39: value 5.26k -> 1k; Mouser Part Number 71-CRCW04025K23FKEDC -> (none)
- R40: value 910k -> 1k; Mouser Part Number 594-MCS04020D9101BE0 -> (none)
- R41: value 1.5k -> 1k; Mouser Part Number 603-RC0402FR-075KL -> (none)
- SW2: footprint tactile_button:TL1030AF200AQJ -> tactile_button:TL1030AF160BQJ
- renumbered C6 to C25, C7 to C26, C8 to C27, C9 to C28, C10 to C29, C12 to C31, C13 to C32, C14 to C33, C15 to C34, C16 to C35, C19 to C37, C20 to C38, C18 to C39, R3 to R42, R2 to R43
Connections:
- net ADC_IN0 is gone; now on net ADC_IN1: IC3.25 (PA3)
- net LNA_OUT_3 is gone; now on net LED_2: R40.1
- net ADC_IN1: no longer IC3.24 (PA2)
- net ADC_IN2: now also IC3.24 (PA2); no longer IC3.23 (PA1)
- net ADC_IN3: now also IC3.23 (PA1); no longer IC3.22 (PA0)
- net GND: now also IC3.15 (PC0), J3.1 (Pin_1), D2.1 (K), D3.1 (K), D4.1 (K), J4.3 (Pin_3); no longer J3.4 (Pin_4)
- net GNDA: now also IC3.18 (PC3_C); no longer R41.1
- net MCU_RX: now also J4.1 (Pin_1)
- net MCU_TX: now also J4.2 (Pin_2)
- net at R41.2: now also D4.2 (A)
- net LED_2: now reaches IC3.56 (PD9)
- net LED_1: now reaches IC3.60 (PD13)
- net LED_1: now also R39.1
- net at R39.2: now also D2.2 (A)
- net +3.3V renamed VBAT
- net VBAT: no longer J3.1 (Pin_1)
- net +3.3VA renamed VDDA33
- net PGA_OUT_0: no longer names the net of R40.2
- net PGA_OUT_0: now also D3.2 (A)
- net UART5_RX: no longer names the net of IC3.51 (PB12)
- net UART5_TX renamed LED_3
- net LED_3: now also R41.1
- net USB_OTG_HS_DM: no longer names the net of IC3.70 (PA11)
- net USB_OTG_HS_DP: no longer names the net of IC3.71 (PA12)
- net USB_OTG_HS_ID: no longer names the net of IC3.69 (PA10)
- new net VIN_SWT: J3.4 (Pin_4)
- new net VREF: IC3.22 (PA0)
- no-connect marks 106 -> 64
Other:
- added sheet Analog Front End (afe.kicad_sch)
- added sheet External Flash (flash.kicad_sch)
- added sheet Power Supply (supply.kicad_sch)
- added sheet Wireless Circuit (wireless.kicad_sch)
- note removed: "--------"
- note removed: "---------------"
- note removed: "0"
- note removed: "1"
- note removed: "1 + RF/RG = 500 RG = 1.5k RF = 750k"
- note removed: "Band-Pass 6 poles"
- note removed: "Band-Pass Filter"
- note removed: "Bootstrapping"
- note removed: "EEG Filtering Stages"
- note removed: "External Flash"
- note removed: "GPIO8"
- note removed: "GPIO9"
- note removed: "Gain = 10 RG = 100k/(Gain - 1) = 11.111k"
- note removed: "Gain = 20 RG = 100k/(Gain - 1) = 5.263k"
- note removed: "High-Pass Filter fc = 1/2πRC"
- note removed: "Low Noise Amplification"
- note removed: "MODE"
- note removed: "Power Supply"
- note removed: "SERIAL"
- note removed: "SPI FLASH"
- note removed: "Variable Gain Amplification"
- note removed: "Wireless Communication"
- note removed: "X"
- note removed: "| |"
- note removed: "| | | |"
- moved on the sheet: C25, C26, C27, C28, C29, C30, C31, C32, C33, C34, C35, C36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

Commit message: Final Hardware Implementation
Parts:
- removed C36: 4.7uF, Capacitor_SMD:C_0603_1608Metric, symbol Device:C
- removed J3: ST-Link, Connector_PinHeader_2.54mm:PinHeader_1x04_P2.54mm_Vertical, symbol Connector_Generic:Conn_01x04
- added J2: Conn_01x05, Connector_PinHeader_2.54mm:PinHeader_1x05_P2.54mm_Vertical, symbol Connector_Generic:Conn_01x05
- C30: value 10uF -> 4.7uF
Connections:
- net BOOT: now also SW2.4; no longer SW2.2
- net GND: now also J2.1 (Pin_1)
- net SWCLK: now also J2.2 (Pin_2)
- net SWDIO: now also J2.3 (Pin_3)
- net SWO: now reaches IC3.89 (PB3)
- net SWO: now also J2.4 (Pin_4)
- net at SW2.1: no longer R42.1
- net VBAT renamed VDD33
- net VDD33: now also J2.5 (Pin_5); no longer C33.1, C34.1, IC3.48 (VCAP_1), IC3.73 (VCAP_2)
- new net: R42.1, SW2.2
- new net VCAP: C33.1, C34.1, IC3.48 (VCAP_1), IC3.73 (VCAP_2)
- no-connect marks 64 -> 63
Other:
- moved on the sheet: C35, R42, R43, SW2
