File: hardware/afe.kicad_sch (KiCad schematic)
At the start: 94 parts, among them IC4 OPA333AIDCKRG4, U1 INA333xxDRG, U10 OPA333xxDCK, U11 MCP602, U12 MCP602, U17 OPA333xxDCK, U18 OPA333xxDCK, U19 OPA333xxDCK, U2 OPA333xxDCK, U3 MCP602, U4 MCP602, U5 INA333xxDRG, U6 OPA333xxDCK, U7 MCP602, U8 MCP602, U9 INA333xxDRG

Commit message: Final Hardware Implementation
Parts:
- R1, R2: value 10k -> 1M
- R15, R3: value 5.26k -> 2.04k
- R27: value 5.26k -> 2.04k; Mouser Part Number 71-CRCW04025K23FKEDC -> 594-MCS04020D9101BE0

Commit message: Interface com FFT
Parts:
- R5: value 1.5k -> 52k
- R6, R8: value 750k -> 1M
- R7: value 1.5k -> 33k
Other:
- note added: "1 + RF/RG = 20"
- note added: "1 + RF/RG = 30"
- note added: "Já está com 1M, e está correto"
- note added: "Trocar para 10nF"
- note added: "Trocar para 620k"
- note added: "Trocar para 680nF"
- note added: "Verificar se pode 270nF"
Changed lines of the file:
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@@
 		)
 	)
-	(text "1 + RF/RG = 250\n\nRG = 3k\nRF = 750k\n\n"
+	(text "1 + RF/RG = 30\n"
 		(exclude_from_sim no)
 		(at 261.366 134.112 0)
@@
 		)
 	)
+	(text "Já está com 1M, e está correto"
+		(exclude_from_sim no)
+		(at 469.392 129.54 0)
+		(effects
+			(font
+				(size 1.27 1.27)
+			)
+		)
+	)
 	(text "Gain = 10\nRG = 100k/(Gain - 1) = 11.111k"
 		(exclude_from_sim no)
@@
 		)
 	)
+	(text "Verificar se pode 270nF\n"
+		(exclude_from_sim no)
+		(at 432.562 102.87 0)
+		(effects
+			(font
+				(size 1.27 1.27)
+			)
+		)
+	)
 	(text "High-Pass Filter \n\nfc = 1/2πRC"
 		(exclude_from_sim no)
@@
 		)
 	)
+	(text "Trocar para 10nF\n"
+		(exclude_from_sim no)
+		(at 369.824 92.71 0)
+		(effects
+			(font
+				(size 1.27 1.27)
+			)
+		)
+	)
 	(text "Gain = 20\nRG = 100k/(Gain - 1) = 5.263k"
 		(exclude_from_sim no)
@@
 		)
 	)
-	(text "1 + RF/RG = 250\n\nRG = 3k\nRF = 750k\n\n"
-		(exclude_from_sim no)
+	(text "1 + RF/RG = 20"
+		(exclude_from_sim yes)
 		(at 223.266 131.572 0)
 		(effects
@@
 		)
 	)
+	(text "Trocar para 10nF\n"
+		(exclude_from_sim no)
+		(at 340.614 122.682 0)
+		(effects
+			(font
+				(size 1.27 1.27)
+			)
+		)
+	)
 	(text "1 + RF/RG = 250\n\nRG = 3k\nRF = 750k\n\n"
 		(exclude_from_sim no)
@@
 		)
 	)
+	(text "Trocar para 680nF"
+		(exclude_from_sim no)
+		(at 447.04 118.11 0)
+		(effects
+			(font
+				(size 1.27 1.27)
+			)
+		)
+	)
+	(text "Trocar para 620k\n"
+		(exclude_from_sim no)
+		(at 344.17 102.87 0)
+		(effects
+			(font
+				(size 1.27 1.27)
+			)
+		)
+	)
 	(text "1 + RF/RG = 250\n\nRG = 3k\nRF = 750k\n\n"
 		(exclude_from_sim no)
@@
 			)
 		)
-		(property "Value" "1.5k"
+		(property "Value" "33k"
 			(at 248.92 130.81 90)
 			(effects
@@
 			)
 		)
-		(property "Value" "750k"
-			(at 220.98 120.65 90)
+		(property "Value" "1M"
+			(at 221.996 120.65 90)
 			(effects
 				(font
@@
 			)
 		)
-		(property "Value" "750k"
-			(at 259.08 123.19 90)
+		(property "Value" "1M"
+			(at 260.096 123.19 90)
 			(effects
 				(font
@@
 			)
 		)
-		(property "Value" "1.5k"
+		(property "Value" "52k"
 			(at 210.82 128.27 90)
 			(effects

Commit message: Hardware v1 final version
Other:
- note added: "Gain = 20 RG = 100k/(Gain - 1) = 2.04k"
Changed lines of the file:
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@@
 		)
 	)
-	(text "Gain = 20\nRG = 100k/(Gain - 1) = 5.263k"
+	(text "Gain = 20\nRG = 100k/(Gain - 1) = 2.04k"
 		(exclude_from_sim no)
-		(at 172.72 132.334 0)
+		(at 173.482 127.762 0)
 		(effects
 			(font
@@
 		(effects
 			(font
-				(size 1.27 1.27)
-			)
-		)
-	)
-	(text "Gain = 10\nRG = 100k/(Gain - 1) = 11.111k"
-		(exclude_from_sim no)
-		(at 172.466 127.508 0)
-		(effects
-			(font
